File: schematics/Samedi/LOA_Samedi.brd (EAGLE design)
At the start: 143.3 x 100 mm, 102 parts, among them IC1 7815, IC10 7806, IC11 7806, IC2 7815, IC3 7815, IC4 7815, IC5 7815, IC6 7815, IC7 7815, IC8 7815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

Commit message: minor change
Routing:
- net L3-2: track 132.5 -> 133.3 mm
Changed lines of the file:
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@@
 <circle x="175.26" y="93.98" radius="2.54" width="0.4064" layer="49"/>
 <wire x1="170.34" y1="0" x2="190.34" y2="0" width="0.4064" layer="49"/>
+<circle x="116.84" y="87.63" radius="3.997959375" width="0" layer="41"/>
+<circle x="106.68" y="87.63" radius="3.997959375" width="0" layer="41"/>
+<circle x="96.52" y="87.63" radius="3.997959375" width="0" layer="41"/>
+<circle x="73.025" y="87.63" radius="3.997959375" width="0" layer="41"/>
+<circle x="53.34" y="87.63" radius="3.997959375" width="0" layer="41"/>
+<circle x="43.18" y="87.63" radius="3.997959375" width="0" layer="41"/>
+<circle x="33.655" y="87.63" radius="3.997959375" width="0" layer="41"/>
+<circle x="23.495" y="87.63" radius="3.997959375" width="0" layer="41"/>
 </plain>
 <attributes>
@@
 <wire x1="68.58" y1="64.516" x2="68.58" y2="62.484" width="0.508" layer="1"/>
 <wire x1="81.788" y1="77.724" x2="68.58" y2="64.516" width="0.508" layer="1"/>
-<wire x1="89.408" y1="77.724" x2="81.788" y2="77.724" width="0.508" layer="1"/>
-<wire x1="96.012" y1="84.328" x2="89.408" y2="77.724" width="0.508" layer="1"/>
-<wire x1="101.6" y1="84.328" x2="96.012" y2="84.328" width="0.508" layer="1"/>
 <wire x1="101.6" y1="84.328" x2="101.6" y2="84.455" width="0.508" layer="1"/>
 <via x="100.076" y="48.26" extent="1-16" drill="0.7" shape="octagon"/>
@@
 <wire x1="101.6" y1="84.455" x2="101.727" y2="84.455" width="0.508" layer="16"/>
 <wire x1="101.727" y1="84.455" x2="104.902" y2="87.63" width="0.508" layer="16"/>
+<wire x1="81.788" y1="77.724" x2="89.154" y2="77.724" width="0.508" layer="1"/>
+<wire x1="89.154" y1="77.724" x2="92.075" y2="80.645" width="0.508" layer="1"/>
+<wire x1="92.075" y1="80.645" x2="98.425" y2="80.645" width="0.508" layer="1"/>
+<wire x1="98.425" y1="80.645" x2="99.695" y2="81.915" width="0.508" layer="1"/>
+<wire x1="99.695" y1="81.915" x2="99.695" y2="83.185" width="0.508" layer="1"/>
+<wire x1="99.695" y1="83.185" x2="100.965" y2="84.455" width="0.508" layer="1"/>
+<wire x1="100.965" y1="84.455" x2="101.6" y2="84.455" width="0.508" layer="1"/>
 </signal>
 <signal name="N$5">
